Commit message: add pose_estimation script with IK service

File: brainswarm_ws/src/roboflex_description/urdf/real_hardware.urdf.xacro (robot description, xacro)
@@ -5,9 +5,9 @@
 <robot
   name="real_robot_hardware">
- <link
+  <link
     name="base_link">
     <inertial>
       <origin
-        xyz="-0.0198856207674204 -0.00141287834695657 0.0217127988880841"
+        xyz="-0.0198856207674204 -0.00141287834695654 0.0217127988880841"
         rpy="0 0 0" />
       <mass
@@ -15,7 +15,7 @@
       <inertia
         ixx="0.000135168968359235"
-        ixy="-6.91009827779043E-06"
-        ixz="-4.27277665593455E-07"
-        iyy="0.000264392316474499"
+        ixy="-6.91009827779041E-06"
+        ixz="-4.27277665593471E-07"
+        iyy="0.0002643923164745"
         iyz="2.33805748764974E-06"
         izz="0.000360228822623865" />
@@ -49,15 +49,15 @@
     <inertial>
       <origin
-        xyz="-0.00073997712798396 -0.00184239661298101 0.0040056795424445"
-        rpy="0 0 0" />
-      <mass
-        value="0.063835393644477" />
-      <inertia
-        ixx="2.05819135406668E-05"
-        ixy="2.15457273252048E-06"
-        ixz="-6.96555382329067E-08"
-        iyy="3.73317819706095E-05"
-        iyz="8.508005425439E-08"
-        izz="3.90116421726318E-05" />
+        xyz="-0.000335711526938457 -0.00195685906883548 0.00400567773618168"
+        rpy="0 0 0" />
+      <mass
+        value="0.0638354178670981" />
+      <inertia
+        ixx="2.04371827614838E-05"
+        ixy="-1.48219694208089E-06"
+        ixz="-8.60140187373712E-08"
+        iyy="3.74765314270289E-05"
+        iyz="6.85161603931178E-08"
+        izz="3.90116575763446E-05" />
     </inertial>
     <visual>
@@ -107,15 +107,15 @@
     <inertial>
       <origin
-        xyz="-0.0220592800955566 -0.0339840872734844 0.0405723636080762"
-        rpy="0 0 0" />
-      <mass
-        value="0.0748071610042354" />
-      <inertia
-        ixx="7.16078709909108E-05"
-        ixy="1.32335423542845E-06"
-        ixz="2.35491971948772E-05"
-        iyy="8.8624298839474E-05"
-        iyz="-9.88088305055191E-07"
-        izz="2.79762099807478E-05" />
+        xyz="-0.0293839678153532 -0.0391750047752968 0.0298252942272988"
+        rpy="0 0 0" />
+      <mass
+        value="0.074807158508353" />
+      <inertia
+        ixx="4.73563804379614E-05"
+        ixy="-5.15954984901729E-06"
+        ixz="3.16484874429079E-05"
+        iyy="8.81011489770943E-05"
+        iyz="4.22015714258333E-06"
+        izz="5.27508477785787E-05" />
     </inertial>
     <visual>
@@ -147,5 +147,5 @@
     type="revolute">
     <origin
-      xyz="0.0040533 0.032246 0.024"
+      xyz="-0.0028235 0.032377 0.024"
       rpy="0 0 0" />
     <parent
@@ -154,5 +154,5 @@
       link="link_2" />
     <axis
-      xyz="0.12444 0.99223 0" />
+      xyz="0.087156 -0.99619 0" />
     <limit
       lower="-1.57"
@@ -165,15 +165,15 @@
     <inertial>
       <origin
-        xyz="0.0396240818912382 -0.0328556511393453 -0.00593954031553318"
-        rpy="0 0 0" />
-      <mass
-        value="0.0758174776124458" />
-      <inertia
-        ixx="4.96269043552773E-05"
-        ixy="-1.7723547111495E-07"
-        ixz="3.04448966068349E-05"
-        iyy="0.000109254251349246"
-        iyz="4.53261122968051E-07"
-        izz="6.91382665468306E-05" />
+        xyz="0.0227758078532524 -0.0328556506617019 0.0329637414290207"
+        rpy="0 0 0" />
+      <mass
+        value="0.075817481422865" />
+      <inertia
+        ixx="4.12901217145756E-05"
+        ixy="-4.85004213224955E-07"
+        ixz="-2.63576710382377E-05"
+        iyy="0.000109254231873346"
+        iyz="4.03948740600622E-08"
+        izz="7.74750349154183E-05" />
     </inertial>
     <visual>
@@ -188,5 +188,5 @@
         name="">
         <color
-          rgba="1 0.549019607843137 0 0.25" />
+          rgba="1 0.549019607843137 0 1" />
       </material>
     </visual>
@@ -205,6 +205,6 @@
     type="revolute">
     <origin
-      xyz="-0.034874 0.0053814 0.0828"
-      rpy="0 0 -0.12476" />
+      xyz="-0.065843 -0.0047567 0.06118"
+      rpy="0 0 0.087266" />
     <parent
       link="link_2" />
@@ -223,15 +223,15 @@
     <inertial>
       <origin
-        xyz="0.0071443767351853 -0.0316783279545622 -0.0228792470549594"
-        rpy="0 0 0" />
-      <mass
-        value="0.0774670735080687" />
-      <inertia
-        ixx="4.69391687400588E-05"
-        ixy="-8.5383245069063E-07"
-        ixz="8.65098318178043E-06"
-        iyy="4.11454270619738E-05"
-        iyz="2.77915843402062E-06"
-        izz="2.20817960680195E-05" />
+        xyz="0.0238071448579615 -0.0316783222787854 0.00277894821163538"
+        rpy="0 0 0" />
+      <mass
+        value="0.0774671928989127" />
+      <inertia
+        ixx="1.97841107265129E-05"
+        ixy="-2.88927123181906E-06"
+        ixz="-3.52790061750793E-06"
+        iyy="4.11454125472179E-05"
+        iyz="-3.23805423941019E-07"
+        izz="4.92368498696563E-05" />
     </inertial>
     <visual>
@@ -263,5 +263,5 @@
     type="revolute">
     <origin
-      xyz="0.087497 0.001 -0.052186"
+      xyz="0.085374 0.001 0.055591"
       rpy="0 0 0" />
     <parent
@@ -281,15 +281,15 @@
     <inertial>
       <origin
-        xyz="0.0227317322742014 -0.0282591595043374 -0.0735491431567077"
-        rpy="0 0 0" />
-      <mass
-        value="0.00458928127195506" />
-      <inertia
-        ixx="2.48457346408623E-07"
-        ixy="1.75608919703415E-09"
-        ixz="-5.74309565861384E-08"
-        iyy="5.92189254891711E-07"
-        iyz="-5.61714965689839E-09"
-        izz="4.14205381701304E-07" />
+        xyz="0.0764884076472838 -0.0289481833034687 0.00870239087002106"
+        rpy="0 0 0" />
+      <mass
+        value="0.00458928127195507" />
+      <inertia
+        ixx="4.2943383442101E-07"
+        ixy="5.8453379790829E-09"
+        ixz="2.32878269343507E-08"
+        iyy="5.92189254891713E-07"
+        iyz="6.84283162314224E-10"
+        izz="2.3322889368892E-07" />
     </inertial>
     <visual>
@@ -339,15 +339,15 @@
     <inertial>
       <origin
-        xyz="0.0227318221834384 -0.0403429519495776 -0.0735494307466795"
+        xyz="0.0764887069201697 -0.0464089888469002 0.00870242590433329"
         rpy="0 0 0" />
       <mass
         value="0.00458915923311391" />
       <inertia
-        ixx="2.48437178254512E-07"
-        ixy="-1.75377298952243E-09"
-        ixz="-5.74288842520944E-08"
-        iyy="5.92150639018822E-07"
-        iyz="5.60974087364876E-09"
-        izz="4.14179232708343E-07" />
+        ixx="4.29407135925781E-07"
+        ixy="-5.83762822506971E-09"
+        ixz="2.3286986618263E-08"
+        iyy="5.92150639018827E-07"
+        iyz="-6.83380621712635E-10"
+        izz="2.33209275037086E-07" />
     </inertial>
     <visual>

File: brainswarm_ws/src/roboflex_description/urdf/roboflex_robotic_arm.urdf.xacro (robot description, xacro)
@@ -409,6 +409,6 @@
         <joint name="joint_1">
             <command_interface name="position">
-                <param name="min">0</param>
-                <param name="max">3.14</param>
+                <param name="min">-1.57</param>
+                <param name="max">1.57</param>
             </command_interface>
             <state_interface name="position">
